File: pcb/macro.kicad_pcb (KiCad board)
At the start: 2 copper layers, 85.5 x 64.2 mm, 21 parts, among them K1 KEYSW, K2 KEYSW, K3 KEYSW, K4 KEYSW, K5 KEYSW, K6 KEYSW, U1 ProMicro

Commit message: generate Gerber file
Other:
- board text added: "lmacro6"
Changed lines of the file:
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@@
       (outputformat 1)
       (mirror false)
-      (drillshape 1)
+      (drillshape 0)
       (scaleselection 1)
-      (outputdirectory "")
+      (outputdirectory "plots")
     )
   )
@@
   (gr_line (start 51.403187 145.125) (end 51.4 85.35) (layer "Edge.Cuts") (width 0.1))
   (gr_line (start 134.7 147.35) (end 53.603187 147.35) (layer "Edge.Cuts") (width 0.1))
+  (gr_text "lmacro6" (at 104.23 95.8) (layer "F.SilkS")
+    (effects (font (size 2 2) (thickness 0.4)))
+  )
   (dimension (type aligned) (layer "Dwgs.User")
     (pts (xy 134.7 147.35) (xy 134.694365 83.15))
@@
   (segment (start 69.37 113.38) (end 62.075 120.675) (width 0.3) (layer "B.Cu") (net 8))
   (segment (start 58.325 120.675) (end 57.025 121.975) (width 0.3) (layer "B.Cu") (net 8))
-  (segment (start 90.49 86.92) (end 93.25 89.68) (width 0.3) (layer "F.Cu") (net 9))
+  (segment (start 89.74 103.18) (end 87.25 103.18) (width 0.3) (layer "F.Cu") (net 9))
+  (segment (start 70.62 86.73) (end 90.3 86.73) (width 0.3) (layer "F.Cu") (net 9))
+  (segment (start 90.3 86.73) (end 93.25 89.68) (width 0.3) (layer "F.Cu") (net 9))
+  (segment (start 63.25 122.43) (end 66.65 119.03) (width 0.3) (layer "F.Cu") (net 9))
+  (segment (start 93.25 99.67) (end 89.74 103.18) (width 0.3) (layer "F.Cu") (net 9))
   (segment (start 66.65 119.03) (end 66.65 90.7) (width 0.3) (layer "F.Cu") (net 9))
-  (segment (start 70.43 86.92) (end 90.49 86.92) (width 0.3) (layer "F.Cu") (net 9))
-  (segment (start 66.65 90.7) (end 70.43 86.92) (width 0.3) (layer "F.Cu") (net 9))
-  (segment (start 89.74 103.18) (end 87.25 103.18) (width 0.3) (layer "F.Cu") (net 9))
-  (segment (start 63.25 122.43) (end 66.65 119.03) (width 0.3) (layer "F.Cu") (net 9))
+  (segment (start 66.65 90.7) (end 70.62 86.73) (width 0.3) (layer "F.Cu") (net 9))
   (segment (start 93.25 89.68) (end 93.25 99.67) (width 0.3) (layer "F.Cu") (net 9))
-  (segment (start 93.25 99.67) (end 89.74 103.18) (width 0.3) (layer "F.Cu") (net 9))
-  (segment (start 64.275 90.065) (end 68.365 85.975) (width 0.3) (layer "F.Cu") (net 10))
-  (segment (start 68.365 85.975) (end 96.955 85.975) (width 0.3) (layer "F.Cu") (net 10))
+  (segment (start 64.275 90.285) (end 68.585 85.975) (width 0.3) (layer "F.Cu") (net 10))
+  (segment (start 64.275 117.29) (end 64.275 90.285) (width 0.3) (layer "F.Cu") (net 10))
+  (segment (start 96.955 85.975) (end 110.57 99.59) (width 0.3) (layer "F.Cu") (net 10))
   (segment (start 110.57 99.59) (end 122.317588 99.59) (width 0.3) (layer "F.Cu") (net 10))
-  (segment (start 96.955 85.975) (end 110.57 99.59) (width 0.3) (layer "F.Cu") (net 10))
+  (segment (start 68.585 85.975) (end 96.955 85.975) (width 0.3) (layer "F.Cu") (net 10))
+  (segment (start 59 122.565) (end 64.275 117.29) (width 0.3) (layer "F.Cu") (net 10))
   (segment (start 122.317588 99.59) (end 125.48 102.752412) (width 0.3) (layer "F.Cu") (net 10))
-  (segment (start 59 122.565) (end 64.275 117.29) (width 0.3) (layer "F.Cu") (net 10))
-  (segment (start 64.275 117.29) (end 64.275 90.065) (width 0.3) (layer "F.Cu") (net 10))
   (segment (start 81.065 104.365) (end 81.065 111.835) (width 0.3) (layer "F.Cu") (net 11))
   (segment (start 77.675 130.885) (end 81.065 130.885) (width 0.3) (layer "F.Cu") (net 11))
